File: battle bunnies.brd (EAGLE design)
At the start: 113 x 33 mm, 44 parts, among them IC1 CP2104, Q1 mmbt2222, Q2 mmbt2222, SW2 KMR2, U1 BME280, U2 SPX3819, U3 MCP73831T-2ACI/OT, X2 ESP32_WROOM32_SKINNY, X4 20329

Commit message: Initial, full, routing - minus Sensors, update gitignore
Parts:
- removed C1, C2: 0.1uF, SparkFun-Capacitors:0603-CAP
- removed D1: MBR120, microbuilder:SOD-123
- removed R11, R13, R14, R17: 4.7K, SparkFun-Resistors:0603-RES
- removed R16: 200, SparkFun-Resistors:0603-RES
- removed SJ4: EN ADR PULLUP, SparkFun-Passives:PAD-JUMPER-3-2OF3_NC_BY_TRACE_YES_SILK_FULL_BOX
- removed U1: BME280, BME280ComponentLibrary:BME280_LGA
- added C9: 10uF, microbuilder:0805-NO
- added JP3: JUMPER-SMT_2_NC_TRACE_SILK, SparkFun-Jumpers:SMT-JUMPER_2_NC_TRACE_SILK
- added Q3: DMG3415U, microbuilder:SOT23-R
- added R12, R7: 100K, microbuilder:0603-NO
- added R9: 10k, SparkFun-Resistors:0603
- D4: value RED -> MBR120; device SparkFun-LED:LED-0603 -> microbuilder:SOD-123
- JP2: device pinhead:1X22 -> SparkFun-Connectors:1X29
- R3: value 10K -> 10k; device microbuilder:RESPACK_4X0603 -> SparkFun-Resistors:0603
- U2: value SPX3819 -> AP2112-3.3
- moved C4 123.7 mm to (102.9, 30.2), turned to 90 degrees
- moved C8 88.9 mm to (102.9, 3.81), turned to 90 degrees
- moved C7 86.1 mm to (100.3, 3.81), turned to 90 degrees
- moved R5 61.9 mm to (109.9, 3.81), flipped to the bottom, turned to 270 degrees
- moved D4 60.5 mm to (17.5, 1.91), flipped to the top, turned to 0 degrees
- moved C5 53.9 mm to (11.3, 18.7)
- moved R3 53.1 mm to (95.6, 30.8), flipped to the bottom, turned to 270 degrees
- moved Q1 52.1 mm to (100.0, 30.5), turned to 180 degrees
- moved R6 50.9 mm to (107.6, 3.81), flipped to the bottom, turned to 270 degrees
- moved Q2 41.6 mm to (92.4, 30.8), flipped to the bottom
- moved JP2 27.9 mm to (1.70, 30.7)
- moved D3 25.1 mm to (96.7, 5.87), turned to 180 degrees
- moved C6 10.9 mm to (19.4, 5.08), turned to 270 degrees
- moved R15 6.65 mm to (18.4, 22.2), flipped to the bottom, turned to 0 degrees
- moved X2 6.55 mm to (106.7, 18.1)
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Connections:
- removed net !CS: R14.1, U1.P$2
- removed net ADC: JP2.21
- removed net CH_PD: JP2.20
- removed net CLK: JP2.12
- removed net CS: JP2.15
- removed net DI: JP2.11
- removed net DO: JP2.14
- removed net GPIO10: JP2.13
- removed net GPIO12/MISO: JP2.17, R11.1, U1.P$3
- removed net GPIO13/MOSI: JP2.16, S2.B2
- removed net GPIO14/SCK: JP2.18, R13.1, U1.P$4
- removed net GPIO15: JP2.9
- removed net GPIO16: JP2.19, S3.B2
- removed net GPIO4/SDA: JP2.6
- removed net GPIO5/SCL: JP2.5
- removed net GPIO9: JP2.10
- removed net IO21: X2.33
- removed net N$11: D4.A
- removed net N$15: R17.1, SJ4.3
- removed net RXD: JP2.4
- removed net SDO/ADR: SJ4.2, U1.P$5
- removed net TXD: IC1.20, JP2.3
- removed net USB_RX: IC1.21
- new net IO23: JP2.17, X2.37
- new net N$6: C5.1, IC1.5, IC1.6, IC1.7, JP3.1
- new net N$7: C6.1, D4.C, Q3.2, R7.2, U2.1
- net 3.3V: now also C9.1, JP3.2; no longer C1.1, C2.1, C5.1, IC1.5, IC1.6, IC1.7, R11.2, R13.2, R14.2, R17.2, U1.P$6, U1.P$8
- net A0_DAC2: now also JP2.25
- net A1_DAC1: now also JP2.24
- net A2_I34: now also JP2.21
- net A3_I39: now also JP2.19
- net A4_IO36: now also JP2.18
- net A5_IO4: now also JP2.8, S2.B2
- net DTR: now also R9.1; no longer R3.4
- net EN: now also JP2.7
- net GND: now also C9.2, JP2.4, JP2.6, R12.1; no longer C1.2, C2.2, R16.2, SJ4.1, U1.P$1, U1.P$7
- net GPIO0: no longer JP2.7
- net GPIO2: now also S3.B2; no longer JP2.8
- net IO12_A11: now also JP2.28
- net IO13_A12: now also JP2.20
- net IO14_A6: now also JP2.27
- net IO15_A8: now also JP2.10
- net IO16: now also JP2.9
- net IO17: now also JP2.11
- net IO27_A10: now also JP2.26
- net IO32_A7: now also JP2.22
- net IO33_A9: now also JP2.23
- net MISO: now also JP2.14
- net MOSI: now also JP2.13
- net N$12: now also R9.2; no longer R3.5
- net N$4: now also R7.1, S1.3; no longer D4.C, R16.1
- net RESET: now also JP2.29; no longer JP2.22
- net RTS: now also R3.1; no longer R3.7
- net RXD0: now also IC1.21
- net SCK: now also JP2.12
- net SCL: now also JP2.16
- net SDA: now also JP2.15, X2.33; no longer X2.37
- net TXD0: now also IC1.20
- net VBAT: now also JP2.5, Q3.3; no longer D1.A
- net VBUS: now also D4.A, JP2.3, Q3.1, R12.2; no longer C6.1, D1.C, S1.3, U2.1
Routing:
- net VBAT: track 0.00 -> 123.8 mm, vias 0 -> 2
- net A5_IO4: track 0.00 -> 114.6 mm, vias 0 -> 6
- net RTS: track 0.00 -> 110.1 mm, vias 0 -> 4
- net TXD0: track 0.00 -> 105.5 mm, vias 0 -> 4
- net RXD0: track 0.00 -> 105.1 mm, vias 0 -> 2
- net DTR: track 0.00 -> 104.6 mm, vias 0 -> 3
- net GPIO2: track 0.00 -> 93.7 mm, vias 0 -> 4
- net IO16: track 0.00 -> 85.5 mm, vias 0 -> 1
- net IO17: track 0.00 -> 83.7 mm, vias 0 -> 1
- net SCL: track 0.00 -> 83.4 mm, vias 0 -> 1
- net IO23: track 0.00 -> 82.6 mm, vias 0 -> 1
- net SCK: track 0.00 -> 81.1 mm, vias 0 -> 1
- net SDA: track 0.00 -> 81.1 mm, vias 0 -> 1
- net MOSI: track 0.00 -> 80.5 mm, vias 0 -> 1
- net MISO: track 0.00 -> 80.5 mm, vias 0 -> 1
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- added copper zone on layer 1, net N$6
- added copper zone on layer 16, net N$8
- added copper zone on layer 1, net RESET
- added copper zone on layer 1, net VBUS
Other:
- board text added: "Disable Serial 3.3V"

Commit message: Mostly Routed - saving and pushing up
Parts:
- added C1, C2: 0.1uF, SparkFun-Capacitors:0603-CAP
- added R11, R13, R14, R17: 4.7K, SparkFun-Resistors:0603-RES
- added SJ4: EN ADR PULLUP, SparkFun-Passives:PAD-JUMPER-3-2OF3_NC_BY_TRACE_YES_SILK_FULL_BOX
- added U4: BMEx80, BME280ComponentLibrary:BME280_LGA
Connections:
- new net !CS: R14.1, U4.P$2
- new net N$15: R17.1, SJ4.3
- new net SDO/ADR: SJ4.2, U4.P$5
- net 3.3V: now also C1.1, C2.1, R11.2, R13.2, R14.2, R17.2, U4.P$6, U4.P$8
- net GND: now also C1.2, C2.2, SJ4.1, U4.P$1, U4.P$7
- net SCL: now also R13.1, U4.P$4
- net SDA: now also R11.1, U4.P$3
Routing:
- net 3.3V: track 0.35 -> 5.86 mm, vias 3 -> 4
- net SCL: track 83.4 -> 88.1 mm
- net !CS: track 0.00 -> 4.46 mm
- net SDA: track 81.1 -> 85.2 mm
- net SDO/ADR: track 0.00 -> 3.18 mm
- net N$15: track 0.00 -> 2.62 mm
Changed lines of the file:
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@@
 <attribute name="NAME" x="12.065" y="23.622" size="0.6096" layer="26" font="vector" ratio="20" rot="MR180" align="bottom-center"/>
+</element>
+<element name="U4" library="BME280ComponentLibrary" package="BME280_LGA" value="BMEx80" x="48.26" y="7.62" smashed="yes">
+<attribute name="PROD_ID" value="IC-13090" x="40.64" y="15.24" size="1.778" layer="27" display="off"/>
+<attribute name="NAME" x="46.355" y="10.16" size="0.8128" layer="25" font="vector"/>
+<attribute name="VALUE" x="48.10125" y="10.16" size="0.8128" layer="27" font="vector"/>
+</element>
+<element name="C1" library="SparkFun-Capacitors" package="0603-CAP" value="0.1uF" x="44.29125" y="9.8425" rot="R180">
+<attribute name="PROD_ID" value="CAP-08604" x="50.64125" y="2.2225" size="1.778" layer="27" rot="R180" display="off"/>
+</element>
+<element name="C2" library="SparkFun-Capacitors" package="0603-CAP" value="0.1uF" x="44.29125" y="7.46125" rot="R180">
+<attribute name="PROD_ID" value="CAP-08604" x="56.99125" y="3.65125" size="1.778" layer="27" rot="R180" display="off"/>
+</element>
+<element name="R11" library="SparkFun-Resistors" package="0603-RES" value="4.7K" x="54.13375" y="6.985" smashed="yes">
+<attribute name="PROD_ID" value="RES-07857" x="47.78375" y="10.795" size="1.778" layer="27" display="off"/>
+<attribute name="NAME" x="51.4985" y="6.7945" size="0.4064" layer="25" font="vector"/>
+<attribute name="VALUE" x="55.8165" y="6.95325" size="0.4064" layer="27" font="vector"/>
+</element>
+<element name="R13" library="SparkFun-Resistors" package="0603-RES" value="4.7K" x="54.13375" y="4.92125" smashed="yes">
+<attribute name="PROD_ID" value="RES-07857" x="41.43375" y="4.92125" size="1.778" layer="27" display="off"/>
+<attribute name="NAME" x="51.4985" y="4.8895" size="0.4064" layer="25" font="vector"/>
+<attribute name="VALUE" x="55.8165" y="4.73075" size="0.4064" layer="27" font="vector"/>
+</element>
+<element name="R14" library="SparkFun-Resistors" package="0603-RES" value="4.7K" x="54.13375" y="9.04875" smashed="yes">
+<attribute name="PROD_ID" value="RES-07857" x="47.78375" y="9.04875" size="1.778" layer="27" display="off"/>
+<attribute name="NAME" x="51.4985" y="9.017" size="0.4064" layer="25" font="vector"/>
+<attribute name="VALUE" x="55.8165" y="9.017" size="0.4064" layer="27" font="vector"/>
+</element>
+<element name="SJ4" library="SparkFun-Passives" package="PAD-JUMPER-3-2OF3_NC_BY_TRACE_YES_SILK_FULL_BOX" value="EN ADR PULLUP" x="47.3075" y="3.4925" rot="R180"/>
+<element name="R17" library="SparkFun-Resistors" package="0603-RES" value="4.7K" x="43.02125" y="3.4925" rot="R180">
+<attribute name="PROD_ID" value="RES-07857" x="60.80125" y="7.3025" size="1.778" layer="27" rot="R180" display="off"/>
 </element>
 </elements>
@@
 <wire x1="107.6325" y1="4.66" x2="105.51" y2="4.66" width="0.4064" layer="16"/>
 <wire x1="105.51" y1="4.66" x2="105.41" y2="4.76" width="0.4064" layer="16"/>
+<contactref element="U4" pad="P$7"/>
+<contactref element="U4" pad="P$1"/>
+<contactref element="C1" pad="2"/>
+<contactref element="C2" pad="2"/>
+<contactref element="SJ4" pad="1"/>
 <wire x1="100.5713" y1="16.51" x2="101.6" y2="16.51" width="0" layer="19" extent="16-16"/>
 <wire x1="103.98" y1="17.7575" x2="101.6" y2="16.51" width="0" layer="19" extent="1-1"/>
@@
 <wire x1="96.52" y1="6.985" x2="96.67875" y2="6.92375" width="0.4064" layer="1"/>
 <contactref element="JP3" pad="2"/>
+<contactref element="U4" pad="P$8"/>
+<contactref element="C2" pad="1"/>
+<contactref element="U4" pad="P$6"/>
+<contactref element="C1" pad="1"/>
+<contactref element="R11" pad="2"/>
+<contactref element="R13" pad="2"/>
+<contactref element="R14" pad="2"/>
+<contactref element="R17" pad="2"/>
+<wire x1="54.98375" y1="4.92125" x2="54.98375" y2="6.985" width="0.8128" layer="1"/>
+<wire x1="54.98375" y1="6.985" x2="54.98375" y2="9.04875" width="0.8128" layer="1"/>
+<wire x1="54.98375" y1="6.985" x2="55.245" y2="6.985" width="0.8128" layer="1"/>
+<wire x1="55.245" y1="6.985" x2="56.03875" y2="6.19125" width="0.8128" layer="1"/>
+<via x="56.03875" y="6.19125" extent="1-16" drill="0.3048"/>
 <wire x1="110.49" y1="26.67" x2="110.49" y2="26.5975" width="0" layer="19" extent="1-1"/>
+<wire x1="47.235" y1="7.295" x2="54.98375" y2="6.985" width="0" layer="19" extent="1-1"/>
+<wire x1="47.235" y1="8.595" x2="47.235" y2="7.295" width="0" layer="19" extent="1-1"/>
+<wire x1="45.14125" y1="7.46125" x2="47.235" y2="7.295" width="0" layer="19" extent="1-1"/>
+<wire x1="45.14125" y1="9.8425" x2="45.14125" y2="7.46125" width="0" layer="19" extent="1-1"/>
+<wire x1="42.17125" y1="3.4925" x2="45.14125" y2="7.46125" width="0" layer="19" extent="1-1"/>
 </signal>
 <signal name="RESET">
@@
 <wire x1="90.17" y1="19.685" x2="50.85625" y2="19.685" width="0.4064" layer="16"/>
 <wire x1="50.85625" y1="19.685" x2="39.795" y2="30.74625" width="0.4064" layer="16"/>
+<contactref element="U4" pad="P$4"/>
+<contactref element="R13" pad="1"/>
+<wire x1="49.285" y1="6.645" x2="51.00875" y2="4.92125" width="0.4064" layer="1"/>
+<wire x1="51.00875" y1="4.92125" x2="53.28375" y2="4.92125" width="0.4064" layer="1"/>
+<wire x1="49.285" y1="6.645" x2="50.85625" y2="19.685" width="0" layer="19" extent="1-16"/>
 </signal>
 <signal name="IO33_A9">
@@
 <wire x1="89.8525" y1="19.05" x2="48.95125" y2="19.05" width="0.4064" layer="16"/>
 <wire x1="48.95125" y1="19.05" x2="37.255" y2="30.74625" width="0.4064" layer="16"/>
+<contactref element="U4" pad="P$3"/>
+<contactref element="R11" pad="1"/>
+<wire x1="49.285" y1="7.295" x2="52.97375" y2="7.295" width="0.4064" layer="1"/>
+<wire x1="52.97375" y1="7.295" x2="53.28375" y2="6.985" width="0.4064" layer="1"/>
+<wire x1="49.285" y1="7.295" x2="48.95125" y2="19.05" width="0" layer="19" extent="1-16"/>
 </signal>
 <signal name="IO14_A6">
@@
 <wire x1="10.16" y1="18.89375" x2="10.16" y2="22.86" width="0.3048" layer="1"/>
 </signal>
+<signal name="!CS">
+<contactref element="U4" pad="P$2"/>
+<contactref element="R14" pad="1"/>
+<wire x1="49.285" y1="7.945" x2="52.18" y2="7.945" width="0.4064" layer="1"/>
+<wire x1="52.18" y1="7.945" x2="53.28375" y2="9.04875" width="0.4064" layer="1"/>
+</signal>
+<signal name="SDO/ADR">
+<contactref element="U4" pad="P$5"/>
+<contactref element="SJ4" pad="2"/>
+<wire x1="47.235" y1="6.645" x2="47.235" y2="3.565" width="0.4064" layer="1"/>
+<wire x1="47.235" y1="3.565" x2="47.3075" y2="3.4925" width="0.4064" layer="1"/>
+</signal>
+<signal name="N$15">
+<contactref element="SJ4" pad="3"/>
+<contactref element="R17" pad="1"/>
+<wire x1="46.4947" y1="3.4925" x2="43.87125" y2="3.4925" width="0.4064" layer="1"/>
+</signal>
 </signals>

Commit message: Big changes - 'final' routing, light sensor, bme280 -> bme680
Parts:
- removed U$31: 18650, Warthog9-Batteries:KEYSTONE1042
- added BT1: LIPO-OUTLINE2000, SparkFun-Batteries:LIPO-2000
- added C10, C11, C12: 1µF, microbuilder:0805-NO@1
- added C13: 2.2µF, microbuilder:0805-NO@1
- added C14, C15, C16, C17, C18: 1uF, SparkFun-Capacitors:0603-CAP
- added D1, D6, D7: MBR0520LT, diode:SOD123
- added J1: (no value), SparkFun-Connectors:JST-2-SMD
- added L1: INDUCTOR-1812-68uH-220ma, SparkFun-Coils:1812
- added Q4: (no value), adafruit:SOT23
- added R16: 2.2, SparkFun-Resistors:0603-RES
- added R18, R19: 10K, microbuilder:0805-NO
- added S4, S5, S6: SWITCH-MOMENTARY-2SMD-4, SparkFun-Electromechanical:TACTILE_SWITCH_TALL
- added U$15: WAVSHARE-BUYDISPLAY-2.132.13-THROUGH, Warthog9-Screens:WAVSHARE-BUYDISPLAY-2.13-THM
- added U1: TSL2591, microbuilder:DFN6_TAOS
- C3, C5, C6, C8, C9: device microbuilder:0805-NO -> microbuilder:0805-NO@1
- C4, C7: device microbuilder:0603-NO -> microbuilder:0603-NO@1
- moved R17 58.5 mm to (99.2, 19.7), turned to 90 degrees
- moved C1 56.7 mm to (98.9, 25.1)
- moved C2 56.7 mm to (98.9, 22.7)
- moved R11 56.7 mm to (108.7, 22.2)
- moved R13 56.7 mm to (108.7, 20.2)
- moved R14 56.7 mm to (108.7, 24.3)
- moved SJ4 56.7 mm to (101.9, 18.7)
- moved U4 56.7 mm to (102.9, 22.9)
- moved D4 36.6 mm to (3.81, 35.9), flipped to the bottom, turned to 90 degrees
- moved R12 33.6 mm to (5.71, 36.8), flipped to the bottom, turned to 90 degrees
- moved C8 29.8 mm to (95.6, 32.7), flipped to the top
- moved C7 29.7 mm to (93.3, 32.7), flipped to the top
- moved C6 28.5 mm to (6.51, 30.5)
- moved Q3 28.4 mm to (8.57, 34.4)
- moved R7 27.9 mm to (3.65, 30.5), turned to 90 degrees
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Connections:
- new net GDR: Q4.1, U$15.2-GDR
- new net N$11: C12.1, D1.C, D6.A
- new net N$14: C12.2, D7.A, L1.1, Q4.3
- new net N$16: C15.1, U$15.18-VDD
- new net N$17: C16.1, U$15.20-VSH
- new net N$18: C17.1, U$15.22-VSL
- new net N$19: C18.1, U$15.24-VCOM
- new net N$20: C14.1, U$15.5-VGH
- new net RESE: Q4.2, R16.1, U$15.3-RESE
- new net VGH: C10.2, D7.C, U$15.21-PREVGH
- new net VGL: C11.2, D1.A, U$15.23-PREVGL
- net 3.3V: now also C13.1, L1.2, R18.2, R19.2, U$15.15-VDDIO, U$15.16-VCI, U1.5
- net A5_IO4: now also U$15.9-BUSY; no longer S2.B2
- net GND: now also C10.1, C11.1, C13.2, C14.2, C15.2, C16.2, C17.2, C18.2, D6.C, J1.1, R16.2, S4.A2, S5.A2, S6.A2, U$15.17-GND, U$15.8-BS1, U1.3; no longer U$31.NEG
- net IO13_A12: now also S2.B2
- net IO14_A6: now also S4.B2
- net IO16: now also U$15.10-RES#
- net IO17: now also U$15.11-D/C#
- net IO23: now also U$15.14-D1
- net IO32_A7: now also S6.B2
- net IO33_A9: now also S5.B2
- net MOSI: now also U$15.13-D0
- net SCK: now also U$15.12-CS#
- net SCL: now also R19.1, U1.1
- net SDA: now also R18.1, U1.6
- net VBAT: now also J1.2; no longer U$31.POS
Routing:
- net IO14_A6: track 32.4 -> 108.3 mm, vias 1 -> 3
- net IO13_A12: track 47.7 -> 117.9 mm, vias 1 -> 3
- net IO32_A7: track 53.8 -> 121.9 mm, vias 1 -> 3
- net IO33_A9: track 49.2 -> 109.7 mm, vias 1 -> 3
- net IO23: track 82.6 -> 120.4 mm, vias 1 -> 2
- net MOSI: track 80.5 -> 111.7 mm, vias 1 -> 3
- net SDA: track 85.2 -> 113.7 mm, vias 1 -> 4
- net SCK: track 81.1 -> 109.5 mm, vias 1 -> 3
- net N$11: track 0.00 -> 27.4 mm, vias 0 -> 3
- net IO17: track 83.7 -> 107.8 mm, vias 1 -> 3
- net IO16: track 85.5 -> 109.0 mm, vias 1 -> 3
- net N$16: track 0.00 -> 21.4 mm, vias 0 -> 2
- net SCL: track 88.1 -> 108.8 mm, vias 1 -> 3
- net N$20: track 0.00 -> 18.9 mm
- net N$17: track 0.00 -> 16.9 mm, vias 0 -> 2
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- added copper zone on layer 1, net 3.3V
- added copper zone on layer 1, net A13_I35
- added copper zone on layer 16, net N$14
- added copper zone on layer 16, net N$7
- added copper zone on layer 1, net SDA
- added copper zone on layer 16, net SDA
- removed copper zone on layer 16, net N$8
- removed copper zone on layer 1, net VBUS
Other:
- board size 113 x 33 mm -> 113 x 59.7 mm
