File: battle bunnies.sch (EAGLE design)
At the start: 40 parts, among them IC1 CP2104, Q1 mmbt2222, Q2 mmbt2222, Q3 DMG3415U, SW2 KMR2, U2 AP2112-3.3, U3 MCP73831T-2ACI/OT, X2 ESP32_WROOM32_SKINNY, X4 20329

Commit message: Mostly Routed - saving and pushing up
Parts:
- added C1, C2: 0.1uF, SparkFun-Capacitors:0.1UF-25V-5%(0603)
- added R11, R13, R14, R17: 4.7K, SparkFun-Resistors:4.7KOHM-1/10W-1%(0603)
- added SJ4: EN ADR PULLUP, SparkFun-Passives:JUMPER-PAD-3-2OF3_NC_BY_TRACE_SMALL
- added U4: BMEx80, BME280ComponentLibrary:BME280
Connections:
- new net !CS: R14.1, U4.!CS
- new net N$15: R17.1, SJ4.3
- new net SDO/ADR: SJ4.2, U4.SDO/ADR
- net 3.3V: now also C1.1, C2.1, R11.2, R13.2, R14.2, R17.2, U4.VDD, U4.VDDIO
- net GND: now also C1.2, C2.2, SJ4.1, U4.GND1, U4.GND2
- net SCL: now also R13.1, U4.SCK/SCL
- net SDA: now also R11.1, U4.SDI/SDA
Other:
- note added: "BME280 - Temp, Humidity BME680 - Temp, Humidity, Pressure, Particle"
- note added: "BMEx80"
- note added: "SJ4 controls the lowest bit of the I2C address--can be: 0x1110110 0x1110111 Open for SPI 3-wire mode"
Changed lines of the file:
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@@
 <part name="R9" library="SparkFun-Resistors" deviceset="10KOHM" device="-0603-1/10W-1%" value="10k"/>
 <part name="JP3" library="SparkFun-Jumpers" deviceset="JUMPER-SMT_2_NC_TRACE" device="_SILK"/>
+<part name="U4" library="BME280ComponentLibrary" deviceset="BME280" device="" value="BMEx80"/>
+<part name="GND1" library="SparkFun-Aesthetics" deviceset="GND" device=""/>
+<part name="GND4" library="SparkFun-Aesthetics" deviceset="GND" device=""/>
+<part name="SUPPLY1" library="SparkFun-Aesthetics" deviceset="3.3V" device=""/>
+<part name="SUPPLY2" library="SparkFun-Aesthetics" deviceset="3.3V" device=""/>
+<part name="GND8" library="SparkFun-Aesthetics" deviceset="GND" device=""/>
+<part name="GND9" library="SparkFun-Aesthetics" deviceset="GND" device=""/>
+<part name="C1" library="SparkFun-Capacitors" deviceset="0.1UF-25V-5%(0603)" device="" value="0.1uF"/>
+<part name="C2" library="SparkFun-Capacitors" deviceset="0.1UF-25V-5%(0603)" device="" value="0.1uF"/>
+<part name="SUPPLY3" library="SparkFun-Aesthetics" deviceset="3.3V" device=""/>
+<part name="R11" library="SparkFun-Resistors" deviceset="4.7KOHM-1/10W-1%(0603)" device="" value="4.7K"/>
+<part name="R13" library="SparkFun-Resistors" deviceset="4.7KOHM-1/10W-1%(0603)" device="" value="4.7K"/>
+<part name="R14" library="SparkFun-Resistors" deviceset="4.7KOHM-1/10W-1%(0603)" device="" value="4.7K"/>
+<part name="SJ4" library="SparkFun-Passives" deviceset="JUMPER-PAD-3-2OF3_NC_BY_TRACE" device="_SMALL" value="EN ADR PULLUP"/>
+<part name="R17" library="SparkFun-Resistors" deviceset="4.7KOHM-1/10W-1%(0603)" device="" value="4.7K"/>
+<part name="SUPPLY5" library="SparkFun-Aesthetics" deviceset="3.3V" device=""/>
+<part name="GND10" library="SparkFun-Aesthetics" deviceset="GND" device=""/>
 </parts>
 <sheets>
@@
 In use by internal
 Flash</text>
+<text x="139.7" y="180.34" size="3.81" layer="97">BMEx80</text>
+<text x="206.248" y="184.658" size="1.778" layer="97" align="top-left">SJ4 controls the lowest bit
+of the I2C address--can be:
+  0x1110110
+  0x1110111
+  Open for SPI 3-wire mode</text>
+<text x="139.7" y="172.72" size="1.778" layer="97">BME280 - Temp, Humidity
+BME680 - Temp, Humidity, Pressure, Particle</text>
 </plain>
 <instances>
@@
 <instance part="R9" gate="G$1" x="101.6" y="144.78"/>
 <instance part="JP3" gate="G$1" x="160.02" y="246.38" rot="R90"/>
+<instance part="U4" gate="U1" x="190.5" y="132.08"/>
+<instance part="GND1" gate="1" x="170.18" y="106.68"/>
+<instance part="GND4" gate="1" x="210.82" y="106.68"/>
+<instance part="SUPPLY1" gate="G$1" x="162.56" y="147.32"/>
+<instance part="SUPPLY2" gate="G$1" x="154.94" y="147.32"/>
+<instance part="GND8" gate="1" x="162.56" y="106.68"/>
+<instance part="GND9" gate="1" x="154.94" y="106.68"/>
+<instance part="C1" gate="G$1" x="154.94" y="114.3"/>
+<instance part="C2" gate="G$1" x="162.56" y="114.3"/>
+<instance part="SUPPLY3" gate="G$1" x="220.98" y="162.56"/>
+<instance part="R11" gate="G$1" x="215.9" y="142.24" rot="R90"/>
+<instance part="R13" gate="G$1" x="226.06" y="142.24" rot="R90"/>
+<instance part="R14" gate="G$1" x="236.22" y="142.24" rot="R90"/>
+<instance part="SJ4" gate="G$1" x="147.32" y="124.46" smashed="yes" rot="R180">
+<attribute name="NAME" x="141.097" y="121.92" size="1.778" layer="95" rot="R90"/>
+<attribute name="VALUE" x="143.383" y="121.92" size="1.778" layer="96" rot="R90"/>
+</instance>
+<instance part="R17" gate="G$1" x="147.32" y="137.16" rot="R90"/>
+<instance part="SUPPLY5" gate="G$1" x="147.32" y="147.32"/>
+<instance part="GND10" gate="1" x="147.32" y="106.68"/>
 </instances>
 <busses>
@@
 <junction x="60.96" y="68.58"/>
 </segment>
+<segment>
+<pinref part="U4" gate="U1" pin="GND2"/>
+<wire x1="175.26" y1="134.62" x2="170.18" y2="134.62" width="0.1524" layer="91"/>
+<pinref part="GND1" gate="1" pin="GND"/>
+<wire x1="170.18" y1="134.62" x2="170.18" y2="109.22" width="0.1524" layer="91"/>
+</segment>
+<segment>
+<pinref part="U4" gate="U1" pin="GND1"/>
+<wire x1="205.74" y1="139.7" x2="210.82" y2="139.7" width="0.1524" layer="91"/>
+<pinref part="GND4" gate="1" pin="GND"/>
+<wire x1="210.82" y1="139.7" x2="210.82" y2="109.22" width="0.1524" layer="91"/>
+</segment>
+<segment>
+<pinref part="GND9" gate="1" pin="GND"/>
+<pinref part="C1" gate="G$1" pin="2"/>
+<wire x1="154.94" y1="109.22" x2="154.94" y2="111.76" width="0.1524" layer="91"/>
+</segment>
+<segment>
+<pinref part="GND8" gate="1" pin="GND"/>
+<pinref part="C2" gate="G$1" pin="2"/>
+<wire x1="162.56" y1="109.22" x2="162.56" y2="111.76" width="0.1524" layer="91"/>
+</segment>
+<segment>
+<pinref part="GND10" gate="1" pin="GND"/>
+<pinref part="SJ4" gate="G$1" pin="1"/>
+<wire x1="147.32" y1="109.22" x2="147.32" y2="119.38" width="0.1524" layer="91"/>
+</segment>
 </net>
 <net name="TXLED" class="0">
@@
 <wire x1="160.02" y1="259.08" x2="160.02" y2="251.46" width="0.1524" layer="91"/>
 </segment>
+<segment>
+<pinref part="SUPPLY1" gate="G$1" pin="3.3V"/>
+<wire x1="162.56" y1="147.32" x2="162.56" y2="139.7" width="0.1524" layer="91"/>
+<pinref part="U4" gate="U1" pin="VDD"/>
+<wire x1="162.56" y1="139.7" x2="175.26" y2="139.7" width="0.1524" layer="91"/>
+<pinref part="C2" gate="G$1" pin="1"/>
+<wire x1="162.56" y1="119.38" x2="162.56" y2="139.7" width="0.1524" layer="91"/>
+<junction x="162.56" y="139.7"/>
+</segment>
+<segment>
+<pinref part="U4" gate="U1" pin="VDDIO"/>
+<wire x1="175.26" y1="129.54" x2="154.94" y2="129.54" width="0.1524" layer="91"/>
+<pinref part="SUPPLY2" gate="G$1" pin="3.3V"/>
+<wire x1="154.94" y1="129.54" x2="154.94" y2="147.32" width="0.1524" layer="91"/>
+<pinref part="C1" gate="G$1" pin="1"/>
+<wire x1="154.94" y1="119.38" x2="154.94" y2="129.54" width="0.1524" layer="91"/>
+<junction x="154.94" y="129.54"/>
+</segment>
+<segment>
+<pinref part="SUPPLY3" gate="G$1" pin="3.3V"/>
+<wire x1="215.9" y1="157.48" x2="215.9" y2="147.32" width="0.1524" layer="91"/>
+<pinref part="R11" gate="G$1" pin="2"/>
+<wire x1="226.06" y1="157.48" x2="226.06" y2="147.32" width="0.1524" layer="91"/>
+<pinref part="R13" gate="G$1" pin="2"/>
+<wire x1="215.9" y1="157.48" x2="220.98" y2="157.48" width="0.1524" layer="91"/>
+<wire x1="220.98" y1="157.48" x2="226.06" y2="157.48" width="0.1524" layer="91"/>
+<wire x1="220.98" y1="162.56" x2="220.98" y2="157.48" width="0.1524" layer="91"/>
+<junction x="220.98" y="157.48"/>
+<pinref part="R14" gate="G$1" pin="2"/>
+<wire x1="236.22" y1="147.32" x2="236.22" y2="157.48" width="0.1524" layer="91"/>
+<wire x1="236.22" y1="157.48" x2="226.06" y2="157.48" width="0.1524" layer="91"/>
+<junction x="226.06" y="157.48"/>
+</segment>
+<segment>
+<pinref part="R17" gate="G$1" pin="2"/>
+<pinref part="SUPPLY5" gate="G$1" pin="3.3V"/>
+<wire x1="147.32" y1="142.24" x2="147.32" y2="147.32" width="0.1524" layer="91"/>
+</segment>
 </net>
 <net name="RESET" class="0">
@@
 <label x="22.86" y="43.18" size="1.778" layer="95"/>
 </segment>
+<segment>
+<pinref part="U4" gate="U1" pin="SCK/SCL"/>
+<wire x1="205.74" y1="124.46" x2="226.06" y2="124.46" width="0.1524" layer="91"/>
+<label x="233.68" y="124.46" size="1.27" layer="95" xref="yes"/>
+<pinref part="R13" gate="G$1" pin="1"/>
+<wire x1="226.06" y1="124.46" x2="233.68" y2="124.46" width="0.1524" layer="91"/>
+<wire x1="226.06" y1="137.16" x2="226.06" y2="124.46" width="0.1524" layer="91"/>
+<junction x="226.06" y="124.46"/>
+</segment>
 </net>
 <net name="IO33_A9" class="0">
@@
 <wire x1="43.18" y1="45.72" x2="22.86" y2="45.72" width="0.1524" layer="91"/>
 <label x="22.86" y="45.72" size="1.778" layer="95"/>
+</segment>
+<segment>
+<pinref part="U4" gate="U1" pin="SDI/SDA"/>
+<wire x1="205.74" y1="129.54" x2="215.9" y2="129.54" width="0.1524" layer="91"/>
+<label x="233.68" y="129.54" size="1.27" layer="95" xref="yes"/>
+<pinref part="R11" gate="G$1" pin="1"/>
+<wire x1="215.9" y1="129.54" x2="233.68" y2="129.54" width="0.1524" layer="91"/>
+<wire x1="215.9" y1="137.16" x2="215.9" y2="129.54" width="0.1524" layer="91"/>
+<junction x="215.9" y="129.54"/>
 </segment>
 </net>
@@
 </segment>
 </net>
+<net name="!CS" class="0">
+<segment>
+<pinref part="U4" gate="U1" pin="!CS"/>
+<wire x1="205.74" y1="134.62" x2="236.22" y2="134.62" width="0.1524" layer="91"/>
+<pinref part="R14" gate="G$1" pin="1"/>
+<wire x1="236.22" y1="137.16" x2="236.22" y2="134.62" width="0.1524" layer="91"/>
+</segment>
+</net>
+<net name="SDO/ADR" class="0">
+<segment>
+<pinref part="U4" gate="U1" pin="SDO/ADR"/>
+<wire x1="175.26" y1="124.46" x2="152.4" y2="124.46" width="0.1524" layer="91"/>
+<pinref part="SJ4" gate="G$1" pin="2"/>
+</segment>
+</net>
+<net name="N$15" class="0">
+<segment>
+<pinref part="SJ4" gate="G$1" pin="3"/>
+<pinref part="R17" gate="G$1" pin="1"/>
+<wire x1="147.32" y1="129.54" x2="147.32" y2="132.08" width="0.1524" layer="91"/>
+</segment>
+</net>

Commit message: Big changes - 'final' routing, light sensor, bme280 -> bme680
Parts:
- removed U$31: 18650, Warthog9-Batteries:18650
- added BT1: LIPO-OUTLINE2000, SparkFun-Batteries:LIPO-OUTLINE2000
- added C10, C11, C12: 1µF, microbuilder:CAP_CERAMIC0805-NOOUTLINE
- added C13: 2.2µF, microbuilder:CAP_CERAMIC0805-NOOUTLINE
- added C14, C15, C16, C17, C18: 1uF, SparkFun-Capacitors:0.1UF-25V-5%(0603)
- added D1, D6, D7: MBR0520LT, diode:MBR0520LT
- added J1: (no value), SparkFun-Connectors:JST_2MM_MALE
- added L1: INDUCTOR-1812-68uH-220ma, SparkFun-Coils:INDUCTOR-1812
- added Q4: (no value), adafruit:MOSFET-NREFLOW
- added R16: 2.2, SparkFun-Resistors:4.7KOHM-1/10W-1%(0603)
- added R18, R19: 10K, microbuilder:RESISTOR0805_NOOUTLINE
- added S4, S5, S6: SWITCH-MOMENTARY-2SMD-4, SparkFun-Electromechanical:SWITCH-MOMENTARY-2SMD-4
- added U$15: WAVSHARE-BUYDISPLAY-2.132.13-THROUGH, Warthog9-Screens:WAVSHARE-BUYDISPLAY-2.132.13-THROUGH
- added U1: TSL2591, microbuilder:LIGHT_TSL2591
Connections:
- new net GDR: Q4.G, U$15.2-GDR
- new net N$11: C12.1, D1.C, D6.A
- new net N$14: C12.2, D7.A, L1.1, Q4.D
- new net N$16: C15.1, U$15.18-VDD
- new net N$17: C16.1, U$15.20-VSH1
- new net N$18: C17.1, U$15.22-VSL
- new net N$19: C18.1, U$15.24-VCOM
- new net N$20: C14.1, U$15.5-VSH2
- new net RESE: Q4.S, R16.1, U$15.3-RESE
- new net VGH: C10.2, D7.C, U$15.21-VGH
- new net VGL: C11.2, D1.A, U$15.23-VGL
- net 3.3V: now also C13.1, L1.2, R18.2, R19.2, U$15.15-VDDIO, U$15.16-VCI, U1.VDD
- net A5_IO4: now also U$15.9-BUSY; no longer S2.2
- net GND: now also C10.1, C11.1, C13.2, C14.2, C15.2, C16.2, C17.2, C18.2, D6.C, J1.-, R16.2, S4.1, S5.1, S6.1, U$15.17-VSS/GND, U$15.8-BS1, U1.GND; no longer U$31.-
- net IO13_A12: now also S2.2
- net IO14_A6: now also S4.2
- net IO16: now also U$15.10-RES#
- net IO17: now also U$15.11-D/C#
- net IO23: now also U$15.14-MOSI
- net IO32_A7: now also S6.2
- net IO33_A9: now also S5.2
- net MOSI: now also U$15.13-SCLK
- net SCK: now also U$15.12-CS#
- net SCL: now also R19.1, U1.SCL
- net SDA: now also R18.1, U1.SDA
- net VBAT: now also J1.+; no longer U$31.+
Other:
- note added: "E-Ink High Voltage Booster"
- note added: "GPIO Table (What's Used, What's Available) ------------------------ GPIO00/Touch1/ADC2_1/CLK01 GPIO01/HS2D1/U0TXD/CLK03 GPIO02/Touch2/ADC2_2/HSPIWP - Button GPIO03/HS2D0/U0RXD/CLK02 GPIO04/Touch0/ADC2_0/HSPIHD - eDSP GPIO05/HS1D6/VSPICS0/(WIRE SPI SS) - eDSP GPIO06/U1CTS/SDCLK/HS1CLK/SPICLK GPIO07/SDD0/HS1D0/SPIQ GPIO08/SDD1/HS1D1/SPI GPIO09/SPIHD/HS1D2/SDD2/U1RXD GPIO10/SPIWP/HS1D3/SDD3/U1TXD GP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"
- note added: "TSL2591 Light Sensor"
- note removed: "GPIO Table (What's Used, What's Available) ------------------------ GPIO00/Touch1/ADC2_1/CLK01 GPIO01/HS2D1/U0TXD/CLK03 GPIO02/Touch2/ADC2_2/HSPIWP - Button GPIO03/HS2D0/U0RXD/CLK02 GPIO04/Touch0/ADC2_0/HSPIHD - Button GPIO05/HS1D6/VSPICS0/(WIRE SPI SS) GPIO06/U1CTS/SDCLK/HS1CLK/SPICLK GPIO07/SDD0/HS1D0/SPIQ GPIO08/SDD1/HS1D1/SPI GPIO09/SPIHD/HS1D2/SDD2/U1RXD GPIO10/SPIWP/HS1D3/SDD3/U1TXD GPIO11/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"
- moved on the sheet: C1, C2, C3, CHG, D3, JP2, R10, R11, R13, R14, R17, R2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
