File: sensornode.brd (EAGLE design)
At the start: 112.3 x 61 mm, 74 parts, among them IC1 CP2104, Q1 mmbt2222, Q2 mmbt2222, Q3 DMG3415U, SW2 KMR2, U1 TSL2591, U2 AP2112-3.3, U3 MCP73831T-2ACI/OT, U4 BMEx80, X2 ESP32_WROOM32_SKINNY, X4 20329

Commit message: Cleaning up a bunch of stuff
Parts:
- added JP1: (no value), pinhead:1X06
Connections:
- net GND: now also JP1.1
- net RXD0: now also JP1.5
- net TXD0: now also JP1.4
Routing:
- net TXD0: track 99.9 -> 113.4 mm
- net RXD0: track 99.3 -> 110.8 mm
Other:
- board size 112.3 x 61 mm -> 112.3 x 63.5 mm
- board text added: "3.3V"
- board text added: ">"
- board text added: "A0 / DAC2"
- board text added: "A1 / DAC1"
- board text added: "BTN / I34"
- board text added: "BTN / IO27"
- board text added: "BTN / IO32"
- board text added: "BTN / IO33"
- board text added: "EBSY / IO4"
- board text added: "ECLK / MOSI"
- board text added: "ECS / SCK"
- board text added: "EDC / IO17"
- board text added: "EMOSI / IO23"
- board text added: "EN"
- board text added: "ERST / IO16"
- board text added: "GND"
- board text added: "HCS / IO15"
- board text added: "HMISO / IO12"
- board text added: "HMOSI / IO13"
- board text added: "HSCLK / IO14"
- board text added: "IO36"
- board text added: "IO39"
- board text added: "MISO"
- board text added: "Off"
- board text added: "On"
- board text added: "RESET"
- board text added: "RX"
- board text added: "SCL"
- board text added: "SDA"
- board text added: "TX"
- board text added: "VBAT"
- board text added: "VBUS"
- board text added: "gnd"
Changed lines of the file:
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@@
 <setting verticaltext="up"/>
 </settings>
-<grid distance="0.1" unitdist="inch" unit="inch" style="lines" multiple="1" display="yes" altdistance="0.00625" altunitdist="inch" altunit="inch"/>
+<grid distance="0.1" unitdist="inch" unit="inch" style="lines" multiple="1" display="yes" altdistance="0.003125" altunitdist="inch" altunit="inch"/>
 <layers>
 <layer number="1" name="Top" color="4" fill="1" visible="yes" active="yes"/>
@@
 <board>
 <plain>
-<wire x1="112.3" y1="0" x2="112.3" y2="61" width="0.1524" layer="20"/>
-<wire x1="112.3" y1="61" x2="0" y2="61" width="0.1524" layer="20"/>
-<wire x1="0" y1="61" x2="0" y2="0" width="0.1524" layer="20"/>
+<wire x1="112.3" y1="0" x2="112.3" y2="63.54" width="0.1524" layer="20"/>
+<wire x1="112.3" y1="63.54" x2="0" y2="63.54" width="0.1524" layer="20"/>
+<wire x1="0" y1="63.54" x2="0" y2="0" width="0.1524" layer="20"/>
 <wire x1="0" y1="0" x2="112.3" y2="0" width="0.1524" layer="20"/>
 <text x="17.93875" y="48.73625" size="0.3048" layer="21">TX LED</text>
@@
 <text x="111.79125" y="4.51" size="0.6096" layer="21" rot="R180">TSL2591
 HDR Light Sensor IR/Full Spectrum</text>
+<text x="1.74625" y="55.40375" size="1.27" layer="21" rot="R315">3.3V</text>
+<text x="4.28625" y="55.40375" size="1.27" layer="21" rot="R315">GND</text>
+<text x="6.82625" y="55.40375" size="1.27" layer="21" rot="R315">VBUS</text>
+<text x="9.36625" y="55.40375" size="1.27" layer="21" rot="R315">GND</text>
+<text x="11.90625" y="55.40375" size="1.27" layer="21" rot="R315">VBAT</text>
+<text x="14.44625" y="55.40375" size="1.27" layer="21" rot="R315">GND</text>
+<text x="16.98625" y="55.40375" size="1.27" layer="21" rot="R315">EN</text>
+<text x="19.52625" y="55.40375" size="1.27" layer="21" rot="R315">EBSY / IO4</text>
+<text x="22.06625" y="55.40375" size="1.27" layer="21" rot="R315">ERST / IO16</text>
+<text x="24.60625" y="55.40375" size="1.27" layer="21" rot="R315">HCS / IO15</text>
+<text x="27.14625" y="55.40375" size="1.27" layer="21" rot="R315">EDC / IO17</text>
+<text x="29.68625" y="55.40375" size="1.27" layer="21" rot="R315">ECS / SCK</text>
+<text x="32.22625" y="55.40375" size="1.27" layer="21" rot="R315">ECLK / MOSI</text>
+<text x="34.925" y="55.40375" size="1.27" layer="21" rot="R315">MISO</text>
+<text x="37.30625" y="55.40375" size="1.27" layer="21" rot="R315">SDA</text>
+<text x="39.84625" y="55.40375" size="1.27" layer="21" rot="R315">SCL</text>
+<text x="42.38625" y="55.40375" size="1.27" layer="21" rot="R315">EMOSI / IO23</text>
+<text x="44.92625" y="55.40375" size="1.27" layer="21" rot="R315">IO36</text>
+<text x="47.46625" y="55.40375" size="1.27" layer="21" rot="R315">IO39</text>
+<text x="50.00625" y="55.40375" size="1.27" layer="21" rot="R315">HMOSI / IO13</text>
+<text x="52.54625" y="55.40375" size="1.27" layer="21" rot="R315">BTN / I34</text>
+<text x="55.08625" y="55.40375" size="1.27" layer="21" rot="R315">BTN / IO32</text>
+<text x="57.62625" y="55.40375" size="1.27" layer="21" rot="R315">BTN / IO33</text>
+<text x="60.16625" y="55.40375" size="1.27" layer="21" rot="R315">A1 / DAC1</text>
+<text x="62.70625" y="55.40375" size="1.27" layer="21" rot="R315">A0 / DAC2</text>
+<text x="65.24625" y="55.245" size="1.27" layer="21" rot="R315">BTN / IO27</text>
+<text x="67.78625" y="55.245" size="1.27" layer="21" rot="R315">HSCLK / IO14</text>
+<text x="70.32625" y="55.08625" size="1.27" layer="21" rot="R315">HMISO / IO12</text>
+<text x="73.025" y="55.08625" size="1.27" layer="21" rot="R315">RESET</text>
+<text x="10.00125" y="61.2775" size="0.8128" layer="21" rot="R45">gnd</text>
+<text x="18.335625" y="61.75375" size="0.8128" layer="21" rot="R45">TX</text>
+<text x="20.875625" y="61.75375" size="0.8128" layer="21" rot="R45">RX</text>
+<text x="10.556875" y="58.816875" size="0.8128" layer="21" rot="R45">&gt;</text>
+<text x="0.47625" y="20.47875" size="1.778" layer="21">On</text>
+<text x="0.47625" y="24.765" size="1.778" layer="21">Off</text>
 </plain>
 <attributes>
@@
 <element name="U$17" library="adafruit" package="MICROSD" value="MICROSD" x="22" y="3" rot="MR90"/>
 <element name="C5" library="microbuilder" package="0805-NO" value="10uF" x="8.09625" y="43.815" rot="R90"/>
+<element name="JP1" library="pinhead" package="1X06" value="" x="18.25625" y="60.80125" smashed="yes">
+<attribute name="NAME" x="26.514425" y="60.40755" size="1.27" layer="25" ratio="10"/>
+<attribute name="VALUE" x="10.63625" y="57.62625" size="1.27" layer="27"/>
+</element>
 </elements>
 <signals>
@@
 <vertex x="113.665" y="21.29"/>
 <vertex x="106.045" y="21.29"/>
-<vertex x="106.045" y="61.595"/>
-<vertex x="0" y="62.23"/>
+<vertex x="106.045" y="64.135"/>
+<vertex x="0" y="64.77"/>
 </polygon>
 <contactref element="X2" pad="15"/>
@@
 <wire x1="39.66845" y1="25.10155" x2="39.37" y2="25.4" width="0.3048" layer="16"/>
 <contactref element="C5" pad="1"/>
+<contactref element="JP1" pad="1"/>
 </signal>
 <signal name="TXLED">
@@
 <vertex x="113.665" y="21.29"/>
 <vertex x="106.045" y="21.29"/>
-<vertex x="106.045" y="61.595"/>
-<vertex x="0" y="62.23"/>
+<vertex x="106.045" y="64.135"/>
+<vertex x="0" y="64.77"/>
 </polygon>
 <contactref element="JP2" pad="1"/>
@@
 <wire x1="78.74" y1="39.37" x2="78.105" y2="40.005" width="0.4064" layer="16"/>
 <wire x1="78.105" y1="40.005" x2="34.29" y2="40.005" width="0.4064" layer="16"/>
-<wire x1="34.29" y1="40.005" x2="23.8125" y2="50.4825" width="0.4064" layer="16"/>
+<wire x1="34.29" y1="40.005" x2="22.86" y2="51.435" width="0.4064" layer="16"/>
 <wire x1="13.21484375" y1="51.117246875" x2="16.192246875" y2="51.117246875" width="0.3048" layer="1"/>
-<wire x1="16.192246875" y1="51.117246875" x2="16.51" y2="51.435" width="0.3048" layer="1"/>
-<via x="16.51" y="51.435" extent="1-16" drill="0.3048"/>
-<wire x1="16.51" y1="51.435" x2="22.86" y2="51.435" width="0.4064" layer="16"/>
-<wire x1="22.86" y1="51.435" x2="23.8125" y2="50.4825" width="0.4064" layer="16"/>
+<via x="19.05" y="51.435" extent="1-16" drill="0.3048"/>
+<wire x1="19.05" y1="51.435" x2="22.86" y2="51.435" width="0.4064" layer="16"/>
+<wire x1="16.192246875" y1="51.117246875" x2="18.732246875" y2="51.117246875" width="0.3048" layer="1"/>
+<wire x1="18.732246875" y1="51.117246875" x2="19.05" y2="51.435" width="0.3048" layer="1"/>
 </signal>
 <signal name="DTR">
@@
 <wire x1="99.742625" y1="35.04565" x2="99.615" y2="35.173275" width="0.4064" layer="1"/>
 <wire x1="99.615" y1="35.173275" x2="99.615" y2="36.2675" width="0.4064" layer="1"/>
+<contactref element="JP1" pad="5"/>
+<wire x1="22.06625" y1="60.80125" x2="23.256875" y2="59.610625" width="0.254" layer="1"/>
+<wire x1="23.256875" y1="59.610625" x2="23.256875" y2="51.196875" width="0.254" layer="1"/>
+<wire x1="23.256875" y1="51.196875" x2="22.225" y2="50.165" width="0.254" layer="1"/>
 </signal>
 <signal name="TXD0">
@@
 <wire x1="100.93315" y1="36.31565" x2="100.93315" y2="34.5185" width="0.4064" layer="1"/>
 <wire x1="100.93315" y1="34.5185" x2="100.8253" y2="34.41065" width="0.4064" layer="1"/>
+<contactref element="JP1" pad="4"/>
+<wire x1="18.176875" y1="51.038125" x2="19.05" y2="50.165" width="0.254" layer="16"/>
+<wire x1="20.955" y1="50.165" x2="19.05" y2="50.165" width="0.254" layer="16"/>
+<wire x1="18.176875" y1="59.451875" x2="19.52625" y2="60.80125" width="0.254" layer="16"/>
+<wire x1="18.176875" y1="51.038125" x2="18.176875" y2="59.451875" width="0.254" layer="16"/>
 </signal>
 <signal name="N$12">

Commit message: Final cleanups going to prototype v2
Routing:
- added copper zone on layer 1, net N$21
- added copper zone on layer 1, net N$22
- added copper zone on layer 16, net N$25
- added copper zone on layer 16, net N$26
- added copper zone on layer 16, net N$27
- added copper zone on layer 16, net N$28
- added copper zone on layer 16, net N$44
Other:
- board text added: "."
- board text added: "A0 / DAC2 / IO26"
- board text added: "A1 / DAC1 / IO25"
- board text added: "BTN / IO34"
- board text added: "ECLK / MOSI / IO18"
- board text added: "ECS / SCK / IO5"
- board text added: "IO2"
- board text added: "IO27"
- board text added: "IO32"
- board text added: "IO33"
- board text added: "IO34"
- board text added: "MISO / IO19"
- board text added: "Reset"
- board text added: "SCL / IO22"
- board text added: "SDA / IO21"
- board text removed: "A0 / DAC2"
- board text removed: "A1 / DAC1"
- board text removed: "BTN / I34"
- board text removed: "ECLK / MOSI"
- board text removed: "ECS / SCK"
- board text removed: "MISO"
- board text removed: "SCL"
- board text removed: "SDA"
Changed lines of the file:
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@@
 <setting verticaltext="up"/>
 </settings>
-<grid distance="0.1" unitdist="inch" unit="inch" style="lines" multiple="1" display="yes" altdistance="0.003125" altunitdist="inch" altunit="inch"/>
+<grid distance="0.1" unitdist="inch" unit="mm" style="lines" multiple="1" display="yes" altdistance="0.003125" altunitdist="inch" altunit="mm"/>
 <layers>
 <layer number="1" name="Top" color="4" fill="1" visible="yes" active="yes"/>
@@
 <text x="17.93875" y="48.73625" size="0.3048" layer="21">TX LED</text>
 <text x="15.875" y="48.895" size="0.3048" layer="21">RX LED</text>
-<text x="107.79125" y="11.51" size="0.6096" layer="21" rot="R180">BME680
+<text x="98.26625" y="10.55625" size="0.4064" layer="21">BME680
 Temp/Humidity/Pressure</text>
 <text x="13.97" y="54.2925" size="0.4064" layer="26" rot="MR270">Disable Serial 3.3V</text>
 <text x="5.715" y="0.3175" size="1.016" layer="21">Sensornode V1.1 | John 'Warthog9' Hawley | (C) 2018 CC-BY-SA 4.0 | https://github.com/unreproducible/sensornode</text>
-<text x="111.79125" y="4.51" size="0.6096" layer="21" rot="R180">TSL2591
+<text x="98.235" y="3.90375" size="0.4064" layer="21">TSL2591
 HDR Light Sensor IR/Full Spectrum</text>
 <text x="1.74625" y="55.40375" size="1.27" layer="21" rot="R315">3.3V</text>
@@
 <text x="24.60625" y="55.40375" size="1.27" layer="21" rot="R315">HCS / IO15</text>
 <text x="27.14625" y="55.40375" size="1.27" layer="21" rot="R315">EDC / IO17</text>
-<text x="29.68625" y="55.40375" size="1.27" layer="21" rot="R315">ECS / SCK</text>
-<text x="32.22625" y="55.40375" size="1.27" layer="21" rot="R315">ECLK / MOSI</text>
-<text x="34.925" y="55.40375" size="1.27" layer="21" rot="R315">MISO</text>
-<text x="37.30625" y="55.40375" size="1.27" layer="21" rot="R315">SDA</text>
-<text x="39.84625" y="55.40375" size="1.27" layer="21" rot="R315">SCL</text>
+<text x="29.68625" y="55.40375" size="1.27" layer="21" rot="R315">ECS / SCK / IO5</text>
+<text x="32.22625" y="55.40375" size="1.27" layer="21" rot="R315">ECLK / MOSI / IO18</text>
+<text x="34.925" y="55.40375" size="1.27" layer="21" rot="R315">MISO / IO19</text>
+<text x="37.30625" y="55.40375" size="1.27" layer="21" rot="R315">SDA / IO21</text>
+<text x="39.84625" y="55.40375" size="1.27" layer="21" rot="R315">SCL / IO22</text>
 <text x="42.38625" y="55.40375" size="1.27" layer="21" rot="R315">EMOSI / IO23</text>
 <text x="44.92625" y="55.40375" size="1.27" layer="21" rot="R315">IO36</text>
 <text x="47.46625" y="55.40375" size="1.27" layer="21" rot="R315">IO39</text>
 <text x="50.00625" y="55.40375" size="1.27" layer="21" rot="R315">HMOSI / IO13</text>
-<text x="52.54625" y="55.40375" size="1.27" layer="21" rot="R315">BTN / I34</text>
+<text x="52.54625" y="55.40375" size="1.27" layer="21" rot="R315">BTN / IO34</text>
 <text x="55.08625" y="55.40375" size="1.27" layer="21" rot="R315">BTN / IO32</text>
 <text x="57.62625" y="55.40375" size="1.27" layer="21" rot="R315">BTN / IO33</text>
-<text x="60.16625" y="55.40375" size="1.27" layer="21" rot="R315">A1 / DAC1</text>
-<text x="62.70625" y="55.40375" size="1.27" layer="21" rot="R315">A0 / DAC2</text>
+<text x="60.16625" y="55.40375" size="1.27" layer="21" rot="R315">A1 / DAC1 / IO25</text>
+<text x="62.70625" y="55.40375" size="1.27" layer="21" rot="R315">A0 / DAC2 / IO26</text>
 <text x="65.24625" y="55.245" size="1.27" layer="21" rot="R315">BTN / IO27</text>
 <text x="67.78625" y="55.245" size="1.27" layer="21" rot="R315">HSCLK / IO14</text>
@@
 <text x="20.875625" y="61.75375" size="0.8128" layer="21" rot="R45">RX</text>
 <text x="10.556875" y="58.816875" size="0.8128" layer="21" rot="R45">&gt;</text>
-<text x="0.47625" y="20.47875" size="1.778" layer="21">On</text>
-<text x="0.47625" y="24.765" size="1.778" layer="21">Off</text>
+<text x="0.238125" y="19.605625" size="1.778" layer="21">On</text>
+<text x="0.47625" y="25.638125" size="1.778" layer="21">Off</text>
+<text x="97.31375" y="1.984375" size="1.016" layer="22" rot="MR0">Sensornode V1.1 | John 'Warthog9' Hawley | (C) 2018 CC-BY-SA 4.0 | https://github.com/unreproducible/sensornode</text>
+<text x="15.478125" y="26.908125" size="1.016" layer="21">IO33</text>
+<text x="25.320625" y="12.3825" size="1.016" layer="21" rot="R90">IO34</text>
+<text x="16.589375" y="12.303125" size="1.016" layer="21" rot="R90">IO32</text>
+<text x="8.651875" y="12.303125" size="1.016" layer="21" rot="R90">IO2</text>
+<text x="15.5575" y="4.92125" size="1.016" layer="21">IO27</text>
+<text x="101.996875" y="16.906875" size="2.54" layer="21">.</text>
+<text x="103.425625" y="60.086875" size="0.6096" layer="21">Reset</text>
 </plain>
 <attributes>
@@
 <via x="20.955" y="50.165" extent="1-16" drill="0.3048"/>
 <wire x1="20.955" y1="50.165" x2="20.955" y2="50.8" width="0.3048" layer="1"/>
-<wire x1="20.955" y1="50.8" x2="18.415" y2="53.34" width="0.3048" layer="1"/>
-<wire x1="18.415" y1="53.34" x2="13.97" y2="53.34" width="0.3048" layer="1"/>
-<wire x1="13.97" y1="53.34" x2="12.71484375" y2="52.08484375" width="0.3048" layer="1"/>
 <wire x1="12.71484375" y1="51.117246875" x2="12.71484375" y2="52.08484375" width="0.3048" layer="1"/>
 <wire x1="100.70465" y1="34.29" x2="100.8253" y2="34.41065" width="0.4064" layer="16"/>
@@
 <wire x1="18.176875" y1="59.451875" x2="19.52625" y2="60.80125" width="0.254" layer="16"/>
 <wire x1="18.176875" y1="51.038125" x2="18.176875" y2="59.451875" width="0.254" layer="16"/>
+<wire x1="12.71484375" y1="52.08484375" x2="13.6525" y2="53.0225" width="0.3048" layer="1"/>
+<wire x1="13.6525" y1="53.0225" x2="18.7325" y2="53.0225" width="0.3048" layer="1"/>
+<wire x1="18.7325" y1="53.0225" x2="20.955" y2="50.8" width="0.3048" layer="1"/>
 </signal>
 <signal name="N$12">
@@
 <wire x1="10.16" y1="47.672090625" x2="9.96484375" y2="47.867246875" width="0.3048" layer="1"/>
 </signal>
+<signal name="N$21">
+<polygon width="0.4064" layer="1">
+<vertex x="13.0175" y="51.7525"/>
+<vertex x="13.0175" y="51.990625"/>
+<vertex x="14.12875" y="53.101875"/>
+<vertex x="18.176875" y="53.101875"/>
+<vertex x="19.52625" y="51.7525"/>
+<vertex x="19.52625" y="51.435"/>
+<vertex x="19.129375" y="51.038125"/>
+<vertex x="13.731875" y="51.038125"/>
+</polygon>
+</signal>
+<signal name="N$22">
+<polygon width="0.3048" layer="1">
+<vertex x="98.58375" y="35.639375"/>
+<vertex x="101.838125" y="35.639375"/>
+<vertex x="101.838125" y="33.099375"/>
+<vertex x="98.7425" y="33.099375"/>
+<vertex x="98.7425" y="35.480625"/>
+</polygon>
+</signal>
+<signal name="N$25">
+<polygon width="0.3048" layer="16" rank="6">
+<vertex x="100.250625" y="35.480625"/>
+<vertex x="104.61625" y="35.480625"/>
+<vertex x="104.61625" y="35.321875"/>
+<vertex x="104.695625" y="35.321875"/>
+<vertex x="104.695625" y="32.385"/>
+<vertex x="104.536875" y="32.385"/>
+<vertex x="101.6" y="29.448125"/>
+<vertex x="101.6" y="33.655"/>
+<vertex x="100.250625" y="35.004375"/>
+</polygon>
+</signal>
+<signal name="N$26">
+<polygon width="0.3048" layer="16" rank="6">
+<vertex x="41.830625" y="18.970625"/>
+<vertex x="48.10125" y="18.970625"/>
+<vertex x="48.5775" y="18.494375"/>
+<vertex x="48.5775" y="13.17625"/>
+<vertex x="49.37125" y="12.3825"/>
+<vertex x="49.37125" y="10.556875"/>
+<vertex x="48.5775" y="9.763125"/>
+<vertex x="48.5775" y="5.794375"/>
+<vertex x="48.021875" y="5.23875"/>
+<vertex x="47.386875" y="5.23875"/>
+<vertex x="42.38625" y="10.239375"/>
+<vertex x="42.38625" y="10.715625"/>
+<vertex x="41.91" y="11.191875"/>
+<vertex x="41.830625" y="11.27125"/>
+</polygon>
+</signal>
+<signal name="N$27">
+<polygon width="0.3048" layer="16" rank="6">
+<vertex x="12.85875" y="7.3025"/>
+<vertex x="12.938125" y="7.381875"/>
+<vertex x="18.57375" y="7.381875"/>
+<vertex x="19.84375" y="8.651875"/>
+<vertex x="19.84375" y="9.286875"/>
+<vertex x="19.3675" y="9.763125"/>
+<vertex x="19.3675" y="22.70125"/>
+<vertex x="31.115" y="34.44875"/>
+<vertex x="49.68875" y="34.44875"/>
+<vertex x="49.768125" y="34.44875"/>
+<vertex x="51.59375" y="32.623125"/>
+<vertex x="51.59375" y="32.0675"/>
+<vertex x="51.514375" y="31.988125"/>
+<vertex x="32.86125" y="31.988125"/>
+<vertex x="27.94" y="27.066875"/>
+<vertex x="22.621875" y="21.74875"/>
+<vertex x="22.621875" y="15.636875"/>
+<vertex x="22.621875" y="10.95375"/>
+<vertex x="21.828125" y="10.16"/>
+<vertex x="20.16125" y="10.16"/>
+<vertex x="20.0025" y="10.00125"/>
+<vertex x="20.0025" y="7.540625"/>
+<vertex x="18.176875" y="5.715"/>
+<vertex x="12.85875" y="5.715"/>
+</polygon>
+</signal>
+<signal name="N$28">
+<polygon width="0.3048" layer="16" rank="6">
+<vertex x="18.415" y="56.276875"/>
+<vertex x="20.0025" y="56.276875"/>
+<vertex x="35.2425" y="41.036875"/>
+<vertex x="33.3375" y="39.131875"/>
+<vertex x="32.385" y="39.131875"/>
+<vertex x="21.11375" y="50.403125"/>
+<vertex x="20.32" y="50.403125"/>
+<vertex x="19.129375" y="50.403125"/>
+<vertex x="18.415" y="51.1175"/>
+<vertex x="18.335625" y="51.1175"/>
+<vertex x="18.335625" y="56.1975" curve="-90"/>
+</polygon>
+</signal>
+<signal name="N$44">
+<polygon width="0.3048" layer="16" rank="6">
+<vertex x="104.14" y="45.72"/>
+<vertex x="87.63" y="45.72"/>
+<vertex x="87.63" y="37.1475"/>
+<vertex x="104.775" y="37.1475"/>
+<vertex x="104.775" y="45.72"/>
+</polygon>
+</signal>
 </signals>
